File: hardware/firethings/ft1.3/raw.kicad_pcb (KiCad board)
At the start: 2 copper layers, 26.7 x 25.4 mm, 17 parts, among them SW1 RESET, SW2 CONFIG, U1 ESP-12, U2 Firethings_Mini, U3 AP2112K

Commit message: Make kicad config more generic
Parts:
- U1: footprint afshar-kicad-libraries:ESP-12-SMD -> firethings-kicad-libs:esp-12-smd
- U2: footprint firethings-mini -> firethings-kicad-libs:firethings-mini
